File: electronics/microcontroller.kicad_sch (KiCad schematic)
At the start: 10 parts, among them J6 Conn_02x03_Counter_Clockwise, U6 MSP430FR2675TRHBT

Commit message: Fixed errors of the first hw prototype
Connections:
- net DALI_RX: now also U6.7 (P1.0_UCB0STE_TA0CLK_A0_VEREF+); no longer U6.11 (P2.2_SYNC_ACLK_COMP0.1)
- net DALI_TX: now also U6.6 (P1.7_UCA0STE_SMCLK_TDO_A7); no longer U6.7 (P1.0_UCB0STE_TA0CLK_A0_VEREF+)
- net VBUF_TEST: now reaches U6.5 (P1.6_UCA0CLK_TA1CLK_TDI_TCLK_A6)
- net LED2: no longer names the net of U6.30 (P2.1_XIN)
Other:
- moved on the sheet: C16, R12, R13, R18
